Commit message: modify urdf/*.xacro更改了官方源码一些不太合理的地方 add meshs/*/v11/*把机械臂新结构文件放进来了 modify README.md添加了一点简单说明

File: urdf/arm/openarm_arm.xacro (robot description, xacro)
@@ -17,6 +17,6 @@
       </joint>
     </xacro:unless>
-    <xacro:link_with_sc no_prefix="${no_prefix}" name="link0" kinematics_link="${kinematics_link}" inertials="${inertials}" reflect="${reflect}"/>
-    <xacro:link_with_sc no_prefix="${no_prefix}" name="link1" kinematics_link="${kinematics_link}" inertials="${inertials}" reflect="${reflect}"/>
+    <xacro:link_with_sc arm_prefix="${arm_prefix}" no_prefix="${no_prefix}" name="link0" kinematics_link="${kinematics_link}" inertials="${inertials}" reflect="${reflect}"/>
+    <xacro:link_with_sc arm_prefix="${arm_prefix}" no_prefix="${no_prefix}" name="link1" kinematics_link="${kinematics_link}" inertials="${inertials}" reflect="${reflect}"/>
     <joint name="${prefix}joint1" type="revolute">
       <xacro:openarm-kinematics name="joint1" config="${kinematics}" reflect="${reflect}"/>
@@ -27,5 +27,5 @@
     </joint>
     <!-- for bimanual offset -->
-    <xacro:link_with_sc no_prefix="${no_prefix}" name="link2" kinematics_link="${kinematics_link}" inertials="${inertials}" reflect="${reflect}"/>
+    <xacro:link_with_sc arm_prefix="${arm_prefix}" no_prefix="${no_prefix}" name="link2" kinematics_link="${kinematics_link}" inertials="${inertials}" reflect="${reflect}"/>
     <xacro:property name="limit_offset_joint2" value="0" />
     <xacro:if value="${prefix.find('right_') != -1}">
@@ -42,5 +42,5 @@
       <xacro:openarm-limits name="joint2" config="${joint_limits}" reflect="${reflect}" offset="${limit_offset_joint2}"/>
     </joint>
-    <xacro:link_with_sc no_prefix="${no_prefix}" name="link3" kinematics_link="${kinematics_link}" inertials="${inertials}" reflect="${reflect}"/>
+    <xacro:link_with_sc arm_prefix="${arm_prefix}" no_prefix="${no_prefix}" name="link3" kinematics_link="${kinematics_link}" inertials="${inertials}" reflect="${reflect}"/>
     <joint name="${prefix}joint3" type="revolute">
       <xacro:openarm-kinematics name="joint3" config="${kinematics}" />
@@ -50,5 +50,5 @@
       <xacro:openarm-limits name="joint3" config="${joint_limits}" />
     </joint>
-    <xacro:link_with_sc no_prefix="${no_prefix}" name="link4" kinematics_link="${kinematics_link}" />
+    <xacro:link_with_sc arm_prefix="${arm_prefix}" no_prefix="${no_prefix}" name="link4" kinematics_link="${kinematics_link}" />
     <joint name="${prefix}joint4" type="revolute">
       <xacro:openarm-kinematics name="joint4" config="${kinematics}" />
@@ -58,5 +58,5 @@
       <xacro:openarm-limits name="joint4" config="${joint_limits}" />
     </joint>
-    <xacro:link_with_sc no_prefix="${no_prefix}" name="link5" kinematics_link="${kinematics_link}" inertials="${inertials}" reflect="${reflect}" />
+    <xacro:link_with_sc arm_prefix="${arm_prefix}" no_prefix="${no_prefix}" name="link5" kinematics_link="${kinematics_link}" inertials="${inertials}" reflect="${reflect}" />
     <joint name="${prefix}joint5" type="revolute">
       <xacro:openarm-kinematics name="joint5" config="${kinematics}" />
@@ -66,5 +66,5 @@
       <xacro:openarm-limits name="joint5" config="${joint_limits}" />
     </joint>
-    <xacro:link_with_sc no_prefix="${no_prefix}" name="link6" kinematics_link="${kinematics_link}" inertials="${inertials}" reflect="${reflect}"/>
+    <xacro:link_with_sc arm_prefix="${arm_prefix}" no_prefix="${no_prefix}" name="link6" kinematics_link="${kinematics_link}" inertials="${inertials}" reflect="${reflect}"/>
     <joint name="${prefix}joint6" type="revolute">
       <xacro:openarm-kinematics name="joint6" config="${kinematics}" />
@@ -74,5 +74,5 @@
       <xacro:openarm-limits name="joint6" config="${joint_limits}" />
     </joint>
-    <xacro:link_with_sc no_prefix="${no_prefix}" name="link7" kinematics_link="${kinematics_link}" inertials="${inertials}" reflect="${reflect}"/>
+    <xacro:link_with_sc arm_prefix="${arm_prefix}" no_prefix="${no_prefix}" name="link7" kinematics_link="${kinematics_link}" inertials="${inertials}" reflect="${reflect}"/>
     <joint name="${prefix}joint7" type="revolute">
       <xacro:openarm-kinematics name="joint7" config="${kinematics}" />

File: urdf/arm/openarm_macro.xacro (robot description, xacro)
@@ -20,5 +20,5 @@
     </xacro:if>
   </xacro:macro>
-  <xacro:macro name="link_with_sc" params="name no_prefix:='false' rpy:='0 0 0' kinematics_link:='' reflect:=1 inertials:=^">
+  <xacro:macro name="link_with_sc" params="name no_prefix:='false' rpy:='0 0 0' kinematics_link:='' reflect:=1 inertials:=^ arm_prefix:=''" >
     <!-- <xacro:property name="prefix" value="${'' if no_prefix else arm_prefix + arm_type + '_'}" /> -->
     <xacro:property name="prefix" value="${'' if no_prefix else 'openarm' + '_' +  arm_prefix}" />

File: urdf/body/openarm_body.xacro (robot description, xacro)
@@ -26,5 +26,6 @@
     name="body_link0"
     no_prefix="${no_prefix}"
-    kinematics_link="${kinematics_link}" />
+    kinematics_link="${kinematics_link}"
+    body_prefix="${body_prefix}" />
     </xacro:macro>
 </robot>

File: urdf/body/openarm_body_macro.xacro (robot description, xacro)
@@ -16,5 +16,5 @@
       </xacro:if>
   </xacro:macro>
-  <xacro:macro name="body_link_with_sc" params="name no_prefix:='false' rpy:='0 0 0' kinematics_link">
+  <xacro:macro name="body_link_with_sc" params="name no_prefix:='false' rpy:='0 0 0' kinematics_link body_prefix:=''" >
     <!-- <xacro:property name="prefix" value="${'' if no_prefix else body_prefix + body_type + '_'}" /> -->
     <xacro:property name="prefix" value="${'' if no_prefix else 'openarm' + '_' + body_prefix}" />
