Commit message: modify urdf/robot/v11.urdf.xacro修正urdf模型各关节的旋转轴与实物初始位相对应,用实测值更新了各个关节的限位区间

File: urdf/robot/v11.urdf.xacro (robot description, xacro)
@@ -73,7 +73,7 @@
     </link>
   </xacro:macro>
-  <xacro:macro name="v11_joint" params="name parent child xyz axis lower upper effort velocity">
+  <xacro:macro name="v11_joint" params="name parent child xyz rpy:='0 0 0' axis lower upper effort velocity">
     <joint name="${name}" type="revolute">
-      <origin xyz="${xyz}" rpy="0 0 0" />
+      <origin xyz="${xyz}" rpy="${rpy}" />
       <parent link="${parent}" />
       <child link="${child}" />
@@ -82,5 +82,5 @@
     </joint>
   </xacro:macro>
-  <xacro:macro name="v11_finger" params="link_name visual_mesh collision_mesh inertial_xyz inertial_rpy mass ixx ixy ixz iyy iyz izz joint_name parent child xyz axis lower upper effort velocity mimic:='none'">
+  <xacro:macro name="v11_finger" params="link_name visual_mesh collision_mesh inertial_xyz inertial_rpy mass ixx ixy ixz iyy iyz izz joint_name parent child xyz rpy:='0 0 0' axis lower upper effort velocity mimic:='none'">
     <xacro:v11_link name="${link_name}"
                     visual_mesh="${visual_mesh}"
@@ -96,5 +96,5 @@
                     izz="${izz}" />
     <joint name="${joint_name}" type="prismatic">
-      <origin xyz="${xyz}" rpy="0 0 0" />
+      <origin xyz="${xyz}" rpy="${rpy}" />
       <parent link="${parent}" />
       <child link="${child}" />
@@ -132,5 +132,5 @@
                     izz="0.000531637742669292" />
     <xacro:v11_joint name="openarm_left_joint1" parent="${v11_root_name}" child="openarm_left_link0"
-             xyz="0.0875 0.00016852 0.31809" axis="-1 0 0" lower="-1.65" upper="3.21" effort="40" velocity="16.754666" />
+             xyz="0.0875 0.00016852 0.31809" axis="-1 0 0" lower="-1.5617" upper="3.1602" effort="40" velocity="16.754666" />
     <xacro:v11_link name="openarm_left_link1"
                     visual_mesh="meshes/arm/v11/visual/left_arm2_Link.stl"
@@ -146,5 +146,5 @@
                     izz="9.02930797233076e-05" />
     <xacro:v11_joint name="openarm_left_joint2" parent="openarm_left_link0" child="openarm_left_link1"
-             xyz="0.067 0.023583 -6.4168e-05" axis="0 1 -0.0028217" lower="-2.89" upper="0.36" effort="40" velocity="16.754666" />
+             xyz="0.067 0.023583 -6.4168e-05" axis="0 -1 0" lower="-0.3099" upper="2.7923" effort="40" velocity="16.754666" />
     <xacro:v11_link name="openarm_left_link2"
                     visual_mesh="meshes/arm/v11/visual/left_arm3_Link.stl"
@@ -160,5 +160,5 @@
                     izz="0.00056421175126219" />
     <xacro:v11_joint name="openarm_left_joint3" parent="openarm_left_link1" child="openarm_left_link2"
-             xyz="-0.0016857 -0.023121 -0.078167" axis="-0.021542 -0.0028211 -0.99976" lower="-3.0" upper="0.13" effort="27" velocity="5.445426" />
+             xyz="-0.0016857 -0.023121 -0.078167" rpy="0 0 1.5708" axis="-0.021542 -0.0028211 -0.99976" lower="-1.5479" upper="1.5084" effort="27" velocity="5.445426" />
     <xacro:v11_link name="openarm_left_link3"
                     visual_mesh="meshes/arm/v11/visual/left_arm4_Link.stl"
@@ -174,5 +174,5 @@
                     izz="0.000100424432052024" />
     <xacro:v11_joint name="openarm_left_joint4" parent="openarm_left_link2" child="openarm_left_link3"
-             xyz="-0.0035655 3.7342e-05 -0.16246" axis="-0.12985 0.99153 0" lower="-0.28" upper="1.63" effort="27" velocity="5.445426" />
+             xyz="-0.0035655 3.7342e-05 -0.16246" rpy="0 0 0" axis="-0.12985 0.99153 0" lower="0" upper="2.393" effort="27" velocity="5.445426" />
     <xacro:v11_link name="openarm_left_link4"
                     visual_mesh="meshes/arm/v11/visual/left_arm5_Link.stl"
@@ -188,5 +188,5 @@
                     izz="0.000182524812032135" />
     <xacro:v11_joint name="openarm_left_joint5" parent="openarm_left_link3" child="openarm_left_link4"
-             xyz="0 0 -0.1049" axis="0 0 -1" lower="-2.58" upper="0.0" effort="7" velocity="20.943946" />
+             xyz="0 0 -0.1049" rpy="0 0 -1.5708" axis="0 0 1" lower="-1.5598" upper="0.9714" effort="7" velocity="20.943946" />
     <xacro:v11_link name="openarm_left_link5"
                     visual_mesh="meshes/arm/v11/visual/left_arm6_Link.stl"
@@ -202,5 +202,5 @@
                     izz="5.65025238376914e-05" />
     <xacro:v11_joint name="openarm_left_joint6" parent="openarm_left_link4" child="openarm_left_link5"
-             xyz="0 0 -0.1205" axis="0 1 0" lower="-0.52" upper="0.52" effort="7" velocity="20.943946" />
+             xyz="0 0 -0.1205" axis="0 1 0" lower="-0.4999" upper="0.4942" effort="7" velocity="20.943946" />
     <xacro:v11_link name="openarm_left_link6"
                     visual_mesh="meshes/arm/v11/visual/left_arm7_Link.stl"
@@ -216,5 +216,5 @@
                     izz="0.0001537900417873" />
     <xacro:v11_joint name="openarm_left_joint7" parent="openarm_left_link5" child="openarm_left_link6"
-             xyz="0.01989 9.503e-05 -0.00064186" axis="0.99948 0 -0.032254" lower="-1.29" upper="1.29" effort="7" velocity="20.943946" />
+             xyz="0.01989 9.503e-05 -0.00064186" axis="-0.99948 0 -0.032254" lower="-1.5222" upper="1.5353" effort="7" velocity="20.943946" />
     <link name="openarm_left_link7" />
     <joint name="openarm_left_link6_to_link7" type="fixed">
@@ -287,5 +287,5 @@
                     izz="0.000530229463662106" />
     <xacro:v11_joint name="openarm_right_joint1" parent="${v11_root_name}" child="openarm_right_link0"
-             xyz="-0.0875000000000191 0.000168522015465328 0.318089913331265" axis="1 0 0" lower="-3.23" upper="1.63" effort="40" velocity="16.754666" />
+             xyz="-0.0875000000000191 0.000168522015465328 0.318089913331265" axis="1 0 0" lower="-3.1514" upper="1.5755" effort="40" velocity="16.754666" />
     <xacro:v11_link name="openarm_right_link1"
                     visual_mesh="meshes/arm/v11/visual/right_arm2_Link.stl"
@@ -301,5 +301,5 @@
                     izz="9.37146230061534e-05" />
     <xacro:v11_joint name="openarm_right_joint2" parent="openarm_right_link0" child="openarm_right_link1"
-             xyz="-0.0670000000000161 0.0228957316518904 0.000442122295684744" axis="0 0.999813609253167 0.0193066504644205" lower="-0.35" upper="2.89" effort="40" velocity="16.754666" />
+             xyz="-0.0670000000000161 0.0228957316518904 0.000442122295684744" axis="0 -0.999813609253167 0.0193066504644205" lower="-2.77" upper="0.3011" effort="40" velocity="16.754666" />
     <xacro:v11_link name="openarm_right_link2"
                     visual_mesh="meshes/arm/v11/visual/right_arm3_Link.stl"
@@ -315,5 +315,5 @@
                     izz="0.000564484880199774" />
     <xacro:v11_joint name="openarm_right_joint3" parent="openarm_right_link1" child="openarm_right_link2"
-             xyz="0.00152231849172751 -0.0213852721731895 -0.0786627305684751" axis="-0.0194545494150194 -0.0193029965330121 0.999624386873342" lower="-3.12" upper="0" effort="27" velocity="5.445426" />
+             xyz="0.00152231849172751 -0.0213852721731895 -0.0786627305684751" rpy="0 0 -1.5708" axis="-0.0194545494150194 -0.0193029965330121 0.999624386873342" lower="-1.6155" upper="1.4586" effort="27" velocity="5.445426" />
     <xacro:v11_link name="openarm_right_link3"
                     visual_mesh="meshes/arm/v11/visual/right_arm4_Link.stl"
@@ -329,5 +329,5 @@
                     izz="9.45252083767826e-05" />
     <xacro:v11_joint name="openarm_right_joint4" parent="openarm_right_link2" child="openarm_right_link3"
-             xyz="0.00316136427993746 0.00363664374112047 -0.162429309541684" axis="0 -0.999813609253167 -0.0193066504644295" lower="-0.24" upper="1.68" effort="27" velocity="5.445426" />
+             xyz="0.00316136427993746 0.00363664374112047 -0.162429309541684" axis="0 1 0" lower="-2.3938" upper="0" effort="27" velocity="5.445426" />
     <xacro:v11_link name="openarm_right_link4"
                     visual_mesh="meshes/arm/v11/visual/right_arm5_Link.stl"
@@ -343,5 +343,5 @@
                     izz="0.000118790406045348" />
     <xacro:v11_joint name="openarm_right_joint5" parent="openarm_right_link3" child="openarm_right_link4"
-             xyz="-0.00746810467908582 0.00202012869338236 -0.104614322597743" axis="0.0711939666374613 -0.0192576596473202 0.997276572300449" lower="-2.58" upper="0.0" effort="7" velocity="20.943946" />
+             xyz="-0.00746810467908582 0.00202012869338236 -0.104614322597743" rpy="0 0 1.5708" axis="0.0711939666374613 -0.0192576596473202 0.997276572300449" lower="-1.5295" upper="1.0009" effort="7" velocity="20.943946" />
     <xacro:v11_link name="openarm_right_link5"
                     visual_mesh="meshes/arm/v11/visual/right_arm6_Link.stl"
@@ -357,5 +357,5 @@
                     izz="5.6499776061088e-05" />
     <xacro:v11_joint name="openarm_right_joint6" parent="openarm_right_link4" child="openarm_right_link5"
-             xyz="-0.00858865089323763 0.00241503877784011 -0.120169304291928" axis="-0.102894166439219 0.994338011479771 0.026546363955051" lower="-0.52" upper="0.52" effort="7" velocity="20.943946" />
+             xyz="-0.00858865089323763 0.00241503877784011 -0.120169304291928" axis="-0.102894166439219 0.994338011479771 0.026546363955051" lower="-0.4746" upper="0.5141" effort="7" velocity="20.943946" />
     <xacro:v11_link name="openarm_right_link6"
                     visual_mesh="meshes/arm/v11/visual/right_arm7_Link.stl"
@@ -371,5 +371,5 @@
                     izz="0.000152150225115048" />
     <xacro:v11_joint name="openarm_right_joint7" parent="openarm_right_link5" child="openarm_right_link6"
-             xyz="-0.0197784297364522 -0.00206652971066514 0.00074375541566038" axis="-0.993890941526293 -0.103845714103361 0.0373746440028857" lower="-1.29" upper="1.29" effort="7" velocity="20.943946" />
+             xyz="-0.0197784297364522 -0.00206652971066514 0.00074375541566038" axis="-0.993890941526293 -0.103845714103361 0.0373746440028857" lower="-1.5725" upper="1.4777" effort="7" velocity="20.943946" />
     <link name="openarm_right_link7" />
     <joint name="openarm_right_link6_to_link7" type="fixed">

Commit message: modify v11.urdf.xacro增加world link,把基座固定在世界坐标系上

File: urdf/robot/v11.urdf.xacro (robot description, xacro)
@@ -480,4 +480,13 @@
     <xacro:v11_head />
   </xacro:unless>
+  <!-- 地面坐标系锚点：world 与机身基座 (body_link0) 重合。
+       真机 / MoveIt / 仿真共用；仿真若需离地高度请在 spawn 时加 -z 偏移，
+       不要在此处修改 world→base 变换。 -->
+  <link name="world" />
+  <joint name="world_to_openarm" type="fixed">
+    <origin xyz="0 0 0.38" rpy="0 0 0" />
+    <parent link="world" />
+    <child link="${v11_root_name}" />
+  </joint>
   <xacro:if value="${ros2_control}">
     <xacro:if value="${bimanual}">
