Commit message: modify v11.urdf.xacro更新新结构的时候把夹爪那部分的关节名和parent修改了,和moveit的srdf和controller.yaml的配置文件对应不上,已修复;modify urdf/ros2_control/openarm.bimanual.ros2_control.xacro 虚拟硬件接口fake_sensor_commands参数弃用了,已修复成mock_sensor_commands

File: urdf/robot/v11.urdf.xacro (robot description, xacro)
@@ -240,5 +240,11 @@
     <xacro:v11_joint name="openarm_left_joint7" parent="openarm_left_link6" child="openarm_left_link7"
              xyz="0.0199 0 0" axis="-1 0 0" lower="-1.56" upper="1.56" effort="7" velocity="20.943946" />
-    <xacro:v11_finger link_name="openarm_left_link8"
+    <link name="openarm_left_hand" />
+    <joint name="openarm_left_hand_joint" type="fixed">
+      <parent link="openarm_left_link7" />
+      <child link="openarm_left_hand" />
+      <origin xyz="0 0 0" rpy="0 0 0" />
+    </joint>
+    <xacro:v11_finger link_name="openarm_left_right_finger"
                       visual_mesh="meshes/ee/openarm_hand_v2/visual/openarm_left_link8.stl"
                       collision_mesh="meshes/ee/openarm_hand_v2/collision/openarm_left_link8.stl"
@@ -252,7 +258,7 @@
                       iyz="2.01335670695175E-05"
                       izz="6.94504322910065E-05"
-                      joint_name="openarm_left_joint8"
-                      parent="openarm_left_link7"
-                      child="openarm_left_link8"
+                      joint_name="openarm_left_finger_joint1"
+                      parent="openarm_left_hand"
+                      child="openarm_left_right_finger"
                       xyz="-0.0205 -0.018499 -0.119"
                       axis="0 -1 0"
@@ -261,5 +267,5 @@
                       effort="7"
                       velocity="20" />
-    <xacro:v11_finger link_name="openarm_left_link9"
+    <xacro:v11_finger link_name="openarm_left_left_finger"
                       visual_mesh="meshes/ee/openarm_hand_v2/visual/openarm_left_link9.stl"
                       collision_mesh="meshes/ee/openarm_hand_v2/collision/openarm_left_link9.stl"
@@ -273,7 +279,7 @@
                       iyz="-2.01356486546468E-05"
                       izz="6.98266910179461E-05"
-                      joint_name="openarm_left_joint9"
-                      parent="openarm_left_link7"
-                      child="openarm_left_link9"
+                      joint_name="openarm_left_finger_joint2"
+                      parent="openarm_left_hand"
+                      child="openarm_left_left_finger"
                       xyz="-0.0205 0.018501 -0.119"
                       axis="0 -1 0"
@@ -282,5 +288,5 @@
                       effort="7"
                       velocity="20"
-                      mimic="openarm_left_joint8" />
+                      mimic="openarm_left_finger_joint1" />
   </xacro:macro>
   <xacro:macro name="v11_arm_right">
@@ -399,5 +405,11 @@
     <xacro:v11_joint name="openarm_right_joint7" parent="openarm_right_link6" child="openarm_right_link7"
              xyz="-0.0199 0 0" axis="-1 0 0" lower="-1.56" upper="1.56" effort="7" velocity="20.943946" />
-    <xacro:v11_finger link_name="openarm_right_link8"
+    <link name="openarm_right_hand" />
+    <joint name="openarm_right_hand_joint" type="fixed">
+      <parent link="openarm_right_link7" />
+      <child link="openarm_right_hand" />
+      <origin xyz="0 0 0" rpy="0 0 0" />
+    </joint>
+    <xacro:v11_finger link_name="openarm_right_right_finger"
                       visual_mesh="meshes/ee/openarm_hand_v2/visual/openarm_right_link8.stl"
                       collision_mesh="meshes/ee/openarm_hand_v2/collision/openarm_right_link8.stl"
@@ -411,7 +423,7 @@
                       iyz="2.01335670836026E-05"
                       izz="6.94504322969539E-05"
-                      joint_name="openarm_right_joint8"
-                      parent="openarm_right_link7"
-                      child="openarm_right_link8"
+                      joint_name="openarm_right_finger_joint1"
+                      parent="openarm_right_hand"
+                      child="openarm_right_right_finger"
                       xyz="0.0205 -0.0185 -0.119"
                       axis="0 -1 0"
@@ -420,5 +432,5 @@
                       effort="7"
                       velocity="20" />
-    <xacro:v11_finger link_name="openarm_right_link9"
+    <xacro:v11_finger link_name="openarm_right_left_finger"
                       visual_mesh="meshes/ee/openarm_hand_v2/visual/openarm_right_link9.stl"
                       collision_mesh="meshes/ee/openarm_hand_v2/collision/openarm_right_link9.stl"
@@ -432,7 +444,7 @@
                       iyz="-2.01356487863785E-05"
                       izz="6.98266910427359E-05"
-                      joint_name="openarm_right_joint9"
-                      parent="openarm_right_link7"
-                      child="openarm_right_link9"
+                      joint_name="openarm_right_finger_joint2"
+                      parent="openarm_right_hand"
+                      child="openarm_right_left_finger"
                       xyz="0.0205 0.0185 -0.119"
                       axis="0 -1 0"
@@ -441,5 +453,5 @@
                       effort="7"
                       velocity="20"
-                      mimic="openarm_right_joint8" />
+                      mimic="openarm_right_finger_joint1" />
   </xacro:macro>
   <xacro:macro name="v11_head">

File: urdf/ros2_control/openarm.bimanual.ros2_control.xacro (robot description, xacro)
@@ -29,5 +29,5 @@
           <xacro:if value="${use_fake_hardware}">
             <plugin>mock_components/GenericSystem</plugin>
-            <param name="fake_sensor_commands">${fake_sensor_commands}</param>
+            <param name="mock_sensor_commands">${fake_sensor_commands}</param>
             <param name="state_following_offset">0.0</param>
           </xacro:if>
@@ -98,5 +98,5 @@
           <xacro:if value="${use_fake_hardware}">
             <plugin>mock_components/GenericSystem</plugin>
-            <param name="fake_sensor_commands">${fake_sensor_commands}</param>
+            <param name="mock_sensor_commands">${fake_sensor_commands}</param>
             <param name="state_following_offset">0.0</param>
           </xacro:if>
